File: PCB/usbhub/usbhub.kicad_pcb (KiCad board)
At the start: 2 copper layers, 35 parts, among them U1 SL2.1S, U2 SL2.1S

Commit message: placement
Parts:
- moved R9 83.0 mm to (171.0, 48.2), turned to -90 degrees
- moved R11 81.6 mm to (161.9, 51.0), turned to -90 degrees
- moved R10 80.4 mm to (164.9, 51.0), turned to -90 degrees
- moved R8 77.2 mm to (171.0, 52.2), turned to 90 degrees
- moved R4 66.7 mm to (171.0, 59.6), turned to -90 degrees
- moved C25 65.6 mm to (169.8, 46.9), turned to 90 degrees
- moved R7 65.3 mm to (171.0, 63.2), turned to 90 degrees
- moved USB7 64.8 mm to (172.6, 73.5), turned to 90 degrees
- moved USB8 63.9 mm to (172.6, 88.5), turned to 90 degrees
- moved U2 62.7 mm to (162.1, 66.3)
- moved C20 62.3 mm to (159.7, 52.5)
- moved C15 59.4 mm to (162.8, 61.7), turned to 180 degrees
- moved USB6 55.7 mm to (174.6, 50.2), turned to 90 degrees
- moved C14 54.9 mm to (166.4, 66.2), turned to -90 degrees
- moved C24 53.0 mm to (169.8, 58.4), turned to 90 degrees
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- renumbered USB1 to usb1_upstream1
Connections:
- net /DN1A renamed /D1A-
- net /DN1B renamed /D1B-
- net /DN2A renamed /D2A-
- net /DN2B renamed /D2B-
- net /DN3A renamed /D3A-
- net /DN3B renamed /D3B-
- net /DN4B renamed /D4B-
- net /DNA renamed /DA-
- net /DNB renamed /DB-
- net /DP1A renamed /D1A+
- net /DP1B renamed /D1B+
- net /DP2A renamed /D2A+
- net /DP2B renamed /D2B+
- net /DP3A renamed /D3A+
- net /DP3B renamed /D3B+
- net /DP4B renamed /D4B+
- net /DPA renamed /DA+
- net /DPB renamed /DB+
Routing:
- added copper zone on B.Cu, net GND
- added copper zone on F.Cu, net GND
Other:
- board outline added: 30.8 x 54.2 mm

Commit message: routing? idk bro
Parts:
- moved C13 1.52 mm to (165.0, 64.7)
- moved C14 1.52 mm to (166.2, 64.7)
- moved C25 1.25 mm to (169.8, 48.2), turned to -90 degrees
- moved R4 0.32 mm to (171.0, 59.2)
Routing:
- net /VBUS: track 0.00 -> 179.0 mm
- net /D4B+: track 0.00 -> 21.5 mm
- net /D4B-: track 0.00 -> 21.3 mm
- net GND: track 0.00 -> 5.39 mm
- net Net-(U1-VDD33): track 0.00 -> 3.03 mm
- net Net-(U2-VDD18): track 0.00 -> 2.89 mm
- net Net-(U1-VDD18): track 0.00 -> 2.73 mm
- net /D3B-: track 0.00 -> 2.64 mm
- net /D3B+: track 0.00 -> 2.61 mm
- net Net-(U2-VDD33): track 0.00 -> 2.40 mm
- net Net-(usb1_upstream1-CC2): track 0.00 -> 1.84 mm
- net Net-(usb1_upstream1-CC1): track 0.00 -> 1.84 mm
- net Net-(USB6-CC1): track 0.00 -> 1.37 mm
- net Net-(USB5-CC1): track 0.00 -> 1.37 mm
- net Net-(USB5-CC2): track 0.00 -> 1.31 mm
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
Commit message: route it lwk
Parts:
- moved C17 4.16 mm to (166.2, 67.5), turned to 90 degrees
- moved C12 4.07 mm to (160.1, 79.0)
- moved C11 3.89 mm to (160.1, 80.2)
- moved C16 3.00 mm to (164.9, 61.0), turned to 0 degrees
- moved C18 2.43 mm to (165.0, 67.5), turned to 90 degrees
- moved C15 2.21 mm to (164.9, 62.2), turned to 0 degrees
- moved C7 1.10 mm to (159.2, 82.0)
- moved C26 1.07 mm to (160.8, 82.0)
- moved C22 1.01 mm to (160.2, 84.0)
- moved C20 1.00 mm to (159.7, 53.5)
- moved U1 0.90 mm to (163.8, 81.8)
- moved C27 0.65 mm to (162.9, 84.8)
- moved C9 0.65 mm to (162.9, 86.0)
- moved U2 0.30 mm to (162.1, 66.0)
Routing:
- net GND: track 5.39 -> 108.3 mm, vias 0 -> 9
- net /DB+: track 0.00 -> 55.3 mm
- net /DB-: track 0.00 -> 55.3 mm
- net /DA+: track 0.00 -> 45.8 mm
- net /DA-: track 0.00 -> 45.8 mm
- net /D1B+: track 0.00 -> 37.0 mm
- net /D1A-: track 0.00 -> 32.0 mm
- net /D1A+: track 0.00 -> 30.5 mm
- net /D1B-: track 0.00 -> 29.6 mm
- net /D3B-: track 2.64 -> 25.0 mm
- net /D3B+: track 2.61 -> 24.9 mm
- net /D2B+: track 0.00 -> 18.8 mm
- net /D2B-: track 0.00 -> 17.8 mm
- net /D2A-: track 0.00 -> 9.70 mm
- net /D3A+: track 0.00 -> 8.73 mm
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Other:
- board size 30.8 x 54.2 mm -> 30.8 x 54.8 mm

Commit message: wow
Routing:
- net /D1B-: track 29.6 -> 36.9 mm
- net GND: track 108.3 -> 107.4 mm

Commit message: some skew tweaks
Routing:
- net GND: track 107.4 -> 102.2 mm
- net /D3A+: track 8.73 -> 9.72 mm
- net /D2B-: track 17.8 -> 18.8 mm
- net /D4B+: track 21.7 -> 22.5 mm
- net /D1A+: track 30.5 -> 31.0 mm
Other:
- board text added: "@jblitzar's usb hub"

Commit message: length match everything nicer
Parts:
- moved R11 0.96 mm to (160.9, 51.0)
Routing:
- net /VBUS: track 184.7 -> 187.3 mm
- net /D2B+: track 18.8 -> 16.5 mm
- net /D2A+: track 8.62 -> 10.5 mm
- net /D2B-: track 18.8 -> 17.2 mm
- net /D3A-: track 8.19 -> 9.68 mm
- net GND: track 102.2 -> 101.3 mm, vias 9 -> 13
- net /D2A-: track 9.70 -> 10.4 mm
- net /D1A+: track 31.0 -> 31.7 mm
- net /D1B-: track 36.9 -> 36.3 mm
